File: coax-probe.sch (KiCad schematic (older format))
At the start: 33 parts, among them J1 Conn_01x02, J2 SMA, J3 Conn_01x02, J4 Conn_01x03, J5 SMA, J6 Conn_01x02, U1 OPA690, U2 INA128, U3 OPA690, U4 CJ431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

Commit message: Try out the LMH6642
Parts:
- removed C13: 100nF, Capacitor_SMD:C_0402_1005Metric, symbol Device:C_Small
- removed R11: 0, Resistor_SMD:R_0603_1608Metric, symbol Device:R_US
- removed R12: DNP, Resistor_SMD:R_0603_1608Metric, symbol Device:R_US
- removed R7: 175, Resistor_SMD:R_0603_1608Metric, symbol Device:R_US
- removed U4: CJ431, Package_TO_SOT_SMD:SOT-23, symbol Reference_Voltage:CJ432
- added C11, C14, C8: 100nF, Capacitor_SMD:C_0402_1005Metric, symbol Device:C_Small
- added C12, C13: 10uF, Capacitor_SMD:C_0805_2012Metric, symbol Device:C
- added U4: ICL7660, Package_SO:SOIC-8_3.9x4.9mm_P1.27mm, symbol Regulator_SwitchedCapacitor:ICL7660
- R1: value 175 -> 510; LCSC C22828 -> C23193
- R2, R3, R8, R9: value 402 -> 510; LCSC C23049 -> C23193
- R6: value 175 -> 0; LCSC C22828 -> C21189
- U1, U3: value OPA690 -> LMH6642; footprint Package_TO_SOT_SMD:TSOT-23-6 -> Package_TO_SOT_SMD:TSOT-23-5; symbol Amplifier_Operational:LMH6611 -> Amplifier_Operational:LMH6609MF; LCSC C206074 -> C779390; MPN OPA690IDBVT -> LMH6642MF/NOPB
Connections:
- net REF is gone; now on net Vref: U2.5 (Ref)
- net GND: now also R6.2, C11.2, C12.1, C14.2, C8.2, U4.3 (GND); no longer U2.4 (V-), U3.2 (V-)
- net INA: now also U3.3 (+); no longer R6.2
- net VCC: now also U1.5 (V+), U3.5 (V+), C14.1, U4.7 (OSC), U4.8 (V+); no longer U1.6 (V+), U3.6 (V+)
- net VSS: now also U2.4 (V-), U3.2 (V-), C11.1, C12.2, C8.1, U4.5 (VOUT)
- net Vref: now reaches R6.1
- net Vref: no longer U3.3 (+)
- new net: C13.1, U4.2 (CAP+)
- new net: C13.2, U4.4 (CAP-)
- no-connect marks 1 -> 2
Other:
- note added: "510ohm protects inputs\nup to 5V from rails."
- note added: "5V-6V"
- note added: "Common mode input range:\nVss-2V - Vcc+2V"
- note added: "Input range up to VCC-1V"
- note added: "TODO: Better output driver, or input dividers to widen effective input common mode range\nMaybe a 3-opamp INA"
- note removed: "175+25 balances 402||402\n\n175 ohm protects inputs up\nto 5V beyond rails."
- note removed: "2.5V Vref shifts input into\nOPA690 common-mode range."
- note removed: "5V-12V"
- note removed: "Common mode input range:\n-2V - VCC+2V"
- note removed: "±3.3V common-mode input\nrange with ±5V supplies."
- moved on the sheet: R1, R2
