File: coax-probe.kicad_pcb (KiCad board)
At the start: 2 copper layers, 28 x 41 mm, 33 parts, among them J1 Conn_01x02, J2 SMA, J3 Conn_01x02, J4 Conn_01x03, J5 SMA, J6 Conn_01x02, U1 OPA690, U2 INA128, U3 OPA690, U4 CJ431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

Commit message: Add power reverse-polarity protection
Parts:
- added Q1: SI2301CDS, Package_TO_SOT_SMD:SOT-23, F.Cu at (177.3, 66.9)
- added Q2: SI2301CDS, Package_TO_SOT_SMD:SOT-23, F.Cu at (177.5, 87.6)
- moved C6 2.90 mm to (177.5, 84.9), turned to 180 degrees
- moved C10 2.61 mm to (177.3, 64.1), turned to 180 degrees
- moved J3 1.50 mm to (180.5, 64.2)
- moved J6 1.50 mm to (180.5, 85.2)
Connections:
- J3 pad 2: VCC -> Net-(J3-Pad2)
- J6 pad 2: VCC -> Net-(J6-Pad2)
Routing:
- net VCC: track 63.1 -> 52.1 mm
- net Net-(J3-Pad2): track 0.00 -> 3.68 mm
- net Net-(J6-Pad2): track 0.00 -> 3.36 mm
